File: c1/v1.1/opac_c1.brd (EAGLE design)
At the start: 49 x 90.9 mm, 77 parts, among them IC2 CP2102, IC3 ATSHA204_SOIC8, IC4 MP1584, IC5 TSC2046QFN, IC6 ATMega-328, IC7 RT9300, IC8 DS1307SO8, Q1 MMBT2222A, Q2 32.768kHz mc306, SW1 PROG, X1 8 MHz

Commit message: Updated opaq n2 schematic and board files.
Parts:
- R20: value 8.2k -> 24k
- R21: value 24k -> 8.2k
Changed lines of the file:
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@@
 <attribute name="VALUE" x="37.932" y="12.211" size="1.27" layer="27" rot="R90"/>
 </element>
-<element name="R20" library="resistor" package="R0603" value="8.2k" x="34.6" y="7" smashed="yes">
+<element name="R20" library="resistor" package="R0603" value="24k" x="34.6" y="7" smashed="yes">
 <attribute name="NAME" x="33.611" y="5.389" size="0.8128" layer="25" ratio="14"/>
 <attribute name="VALUE" x="33.711" y="4.968" size="1.27" layer="27"/>
 </element>
-<element name="R21" library="resistor" package="R0603" value="24k" x="31.2" y="7" smashed="yes">
+<element name="R21" library="resistor" package="R0603" value="8.2k" x="31.2" y="7" smashed="yes">
 <attribute name="NAME" x="30.211" y="5.389" size="0.8128" layer="25" ratio="14"/>
 <attribute name="VALUE" x="30.311" y="4.968" size="1.27" layer="27"/>
