File: c1/v1.1/opac_c1.sch (EAGLE design)
At the start: 77 parts, among them IC2 CP2102, IC3 ATSHA204_SOIC8, IC4 MP1584, IC5 TSC2046QFN, IC6 ATMega-328, IC7 RT9300, IC8 DS1307SO8, Q1 MMBT2222A, Q2 32.768kHz mc306, SW1 PROG, X1 8 MHz

Commit message: Updated opaq n2 schematic and board files.
Parts:
- R20: value 8.2k -> 24k
- R21: value 24k -> 8.2k
Changed lines of the file:
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@@
 <part name="C8" library="resistor" deviceset="C-EU" device="C3216" value="10uf"/>
 <part name="GND14" library="SparkFun" deviceset="GND" device=""/>
-<part name="R20" library="resistor" deviceset="R-EU_" device="R0603" value="8.2k"/>
-<part name="R21" library="resistor" deviceset="R-EU_" device="R0603" value="24k"/>
+<part name="R20" library="resistor" deviceset="R-EU_" device="R0603" value="24k"/>
+<part name="R21" library="resistor" deviceset="R-EU_" device="R0603" value="8.2k"/>
 <part name="GND15" library="SparkFun" deviceset="GND" device=""/>
 <part name="C9" library="resistor" deviceset="C-EU" device="C3216" value="10uf"/>
