File: n1/v2.1/opaq_n1.brd (EAGLE design)
At the start: 30.3 x 50.4 mm, 44 parts, among them IC1 RT9013-XXXB, IC2 TS5A3157, IC3 ATSHA204_SOIC8, IC4 ACS712, IC5 ADS1100, IC6 ATMega-328, IC7 AT25F512BWIDE_5.3MM, IC8 LM2594HV, K1 62101021021, Q1 IRLR3915, Q2 IRLR3915, Q3 IRLR3915, Q4 IRLR3915, X1 16 MHz

Commit message: Small changes of the opaq n1 board.
Parts:
- added SJ1: (no value), SparkFun:SJ_2S-TRACE
- C10: value (none) -> 22uf 50v
- C2: value (none) -> 100uf 10v
- IC7: value AT25F512BWIDE_5.3MM -> AT25HP512
- moved IC1 0.20 mm to (26.9, 19.7)
Connections:
- net +5V: now also SJ1.1
- net 3.3V: now also SJ1.2
Routing:
- net 3.3V: track 17.7 -> 18.8 mm
Other:
- board text added: "Board Version 2.1 14/11/2016"
- board text removed: "Board Version 2.1 28/04/2016"
Changed lines of the file:
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@@
 <wire x1="30.1" y1="47.7" x2="27.6" y2="50.2" width="1.6" layer="46" curve="90"/>
 <text x="11.8" y="-10.1" size="1.778" layer="51">André Pedro</text>
-<text x="1.2" y="2.1" size="0.8128" layer="26" ratio="14" rot="MR90">Board Version 2.1 28/04/2016</text>
+<text x="1.2" y="2.1" size="0.8128" layer="26" ratio="14" rot="MR90">Board Version 2.1 14/11/2016</text>
 </plain>
 <attributes>
@@
 <attribute name="NAME" x="16.167875" y="15.67204375" size="0.6096" layer="25" ratio="14" rot="R270"/>
 </element>
-<element name="IC1" library="v-reg_extra" package="SOT23-5" value="RT9013-XXXB" x="26.9" y="19.9" smashed="yes">
-<attribute name="NAME" x="24.4694625" y="20.664040625" size="0.6096" layer="25" ratio="14" rot="R270"/>
-<attribute name="VALUE" x="24.995" y="16.725" size="0.8128" layer="27" ratio="10"/>
+<element name="IC1" library="v-reg_extra" package="SOT23-5" value="RT9013-XXXB" x="26.9" y="19.7" smashed="yes">
+<attribute name="NAME" x="24.4694625" y="20.464040625" size="0.6096" layer="25" ratio="14" rot="R270"/>
+<attribute name="VALUE" x="24.995" y="16.525" size="0.8128" layer="27" ratio="10"/>
 </element>
 <element name="IC8" library="apedro_lib" package="SO08" value="LM2594HV" x="24.8" y="32.5" smashed="yes">
@@
 <attribute name="VALUE" x="10.343" y="1.984" size="0.4064" layer="27" font="vector" rot="R90"/>
 </element>
-<element name="IC7" library="LowPowerLab" package="SO08WIDE" value="AT25F512BWIDE_5.3MM" x="4.4" y="10.3" smashed="yes">
+<element name="IC7" library="LowPowerLab" package="SO08WIDE" value="AT25HP512" x="4.4" y="10.3" smashed="yes">
 <attribute name="VALUE" x="5.832" y="9.9005" size="0.5" layer="27" ratio="10" rot="R180"/>
 <attribute name="NAME" x="7.07278125" y="11.008240625" size="0.6096" layer="25" ratio="14" rot="R270"/>
@@
 <attribute name="VALUE" x="21.49" y="38.92" size="1.27" layer="27"/>
 </element>
-<element name="C2" library="rcl" package="C/6032-28R" value="" x="25" y="26" smashed="yes">
+<element name="C2" library="rcl" package="C/6032-28R" value="100uf 10v" x="25" y="26" smashed="yes">
 <attribute name="NAME" x="27.3695625" y="27.6472" size="0.8128" layer="25" ratio="14"/>
 <attribute name="VALUE" x="22" y="22.95" size="1.27" layer="27"/>
 </element>
-<element name="C10" library="rcl" package="D/7343-31R" value="" x="23.2" y="38" smashed="yes">
+<element name="C10" library="rcl" package="D/7343-31R" value="22uf 50v" x="23.2" y="38" smashed="yes">
 <attribute name="NAME" x="21.432159375" y="39.997" size="0.8128" layer="25" ratio="14" rot="R90"/>
 <attribute name="VALUE" x="19.55" y="34.425" size="1.27" layer="27"/>
@@
 <attribute name="NAME" x="7.138" y="32.0745" size="0.6096" layer="26" ratio="14" rot="MR180"/>
 <attribute name="VALUE" x="6.884" y="34.297" size="0.4064" layer="28" rot="MR180"/>
+</element>
+<element name="SJ1" library="SparkFun" package="SJ_2S-TRACE" value="" x="26.4" y="23" smashed="yes" rot="R180">
+<attribute name="NAME" x="27.77" y="24.3525" size="0.8128" layer="25" ratio="14" rot="R270"/>
+<attribute name="VALUE" x="27.3525" y="24.651" size="0.4064" layer="27" rot="R180"/>
 </element>
 </elements>
@@
 <wire x1="26" y1="13.2" x2="25.2" y2="13.2" width="0.4064" layer="1"/>
 <wire x1="25.2" y1="13.2" x2="25.1" y2="13.1" width="0.4064" layer="1"/>
-<wire x1="25.95" y1="18.5999" x2="25.1" y2="18.5999" width="0.6096" layer="1"/>
-<wire x1="25.1" y1="18.5999" x2="23.7999" y2="18.5999" width="0.6096" layer="1"/>
+<wire x1="25.1" y1="18.5999" x2="24.9" y2="18.5999" width="0.6096" layer="1"/>
+<wire x1="24.9" y1="18.5999" x2="23.7999" y2="18.5999" width="0.6096" layer="1"/>
 <wire x1="25.1" y1="13.1" x2="25.1" y2="18.5999" width="0.6096" layer="1"/>
 <wire x1="18.5" y1="13.75" x2="18.5" y2="14.6" width="0.254" layer="1"/>
@@
 <wire x1="26.705" y1="29.8838" x2="26.7888" y2="29.8" width="0.4064" layer="1"/>
 <contactref element="C2" pad="+"/>
-<wire x1="25.95" y1="18.5999" x2="25.95" y2="19.75" width="0.6096" layer="1"/>
+<wire x1="25.95" y1="18.3999" x2="25.95" y2="19.75" width="0.6096" layer="1"/>
 <wire x1="25.95" y1="19.75" x2="26.1" y2="19.9" width="0.6096" layer="1"/>
 <wire x1="26.1" y1="19.9" x2="26.8" y2="19.9" width="0.6096" layer="1"/>
@@
 <wire x1="12.35" y1="18.7" x2="12.35" y2="18.1" width="0.254" layer="1"/>
 <wire x1="12.35" y1="18.1" x2="12.15" y2="17.9" width="0.254" layer="1"/>
+<contactref element="SJ1" pad="1"/>
+<wire x1="25.95" y1="18.3999" x2="25.1" y2="18.3999" width="0.6096" layer="1"/>
+<wire x1="25.1" y1="18.3999" x2="24.9" y2="18.5999" width="0.6096" layer="1"/>
+<wire x1="26.9" y1="22.7" x2="26.908" y2="23" width="0" layer="19" extent="1-1"/>
 </signal>
 <signal name="FILT">
@@
 <contactref element="IC1" pad="3"/>
 <contactref element="R4" pad="2"/>
-<wire x1="27.85" y1="18.5999" x2="27.85" y2="16.35" width="0.4064" layer="1"/>
+<wire x1="27.85" y1="18.3999" x2="27.85" y2="16.35" width="0.4064" layer="1"/>
 <wire x1="27.85" y1="16.35" x2="27.8" y2="16.3" width="0.4064" layer="1"/>
 </signal>
@@
 <contactref element="C4" pad="1"/>
 <contactref element="MODULE1" pad="1"/>
-<wire x1="25.95" y1="21.2001" x2="25.95" y2="22.15" width="0.3048" layer="1"/>
-<wire x1="25.95" y1="22.15" x2="25.6" y2="22.5" width="0.3048" layer="1"/>
-<wire x1="25.6" y1="22.5" x2="24.7" y2="22.5" width="0.3048" layer="1"/>
+<wire x1="25.95" y1="21.0001" x2="25.95" y2="22.15" width="0.3048" layer="1"/>
 <via x="20" y="28.5" extent="1-16" drill="0.5"/>
 <wire x1="19.8" y1="27.2" x2="18.8" y2="27.2" width="0.3048" layer="1"/>
@@
 <wire x1="19.8" y1="27.2" x2="19.8" y2="28.3" width="0.3048" layer="1"/>
 <wire x1="19.8" y1="28.3" x2="20" y2="28.5" width="0.3048" layer="1"/>
-<wire x1="20.4" y1="22.5" x2="24.7" y2="22.5" width="0.254" layer="1"/>
+<wire x1="20.4" y1="22.5" x2="24.4" y2="22.5" width="0.254" layer="1"/>
+<contactref element="SJ1" pad="2"/>
+<wire x1="25.2" y1="23" x2="25.892" y2="23" width="0.3048" layer="1"/>
+<wire x1="25.892" y1="23" x2="25.892" y2="22.208" width="0.3048" layer="1"/>
+<wire x1="25.892" y1="22.208" x2="25.95" y2="22.15" width="0.3048" layer="1"/>
+<wire x1="24.4" y1="22.5" x2="24.7" y2="22.5" width="0.3048" layer="1"/>
+<wire x1="24.7" y1="22.5" x2="25.2" y2="23" width="0.3048" layer="1"/>
 </signal>
 <signal name="NRF24_CE">
