File: n1/v2.1/opaq_n1.sch (EAGLE design)
At the start: 44 parts, among them IC1 RT9013-XXXB, IC2 TS5A3157, IC3 ATSHA204_SOIC8, IC4 ACS712, IC5 ADS1100, IC6 ATMega-328, IC7 AT25F512BWIDE_5.3MM, IC8 LM2594HV, K1 62101021021, Q1 IRLR3915, Q2 IRLR3915, Q3 IRLR3915, Q4 IRLR3915, X1 16 MHz

Commit message: Small changes of the opaq n1 board.
Parts:
- added SJ1: SOLDERJUMPERTRACE, SparkFun:SOLDERJUMPERTRACE
- C10: value (none) -> 22uf 50v
- C2: value (none) -> 100uf 10v
- IC7: value AT25F512BWIDE_5.3MM -> AT25HP512
Connections:
- net +5V: now also SJ1.1
- net 3.3V: now also SJ1.2
Other:
- note added: "3.3v Power Supply"
- note added: "ADC"
- note added: "Analog Switch"
- note added: "Crypto Module"
- note added: "Current Sensor"
- note added: "Dimmer Switchers"
- note added: "Flash"
- note added: "MCU"
- note added: "NRF24L01+ Module"
- note added: "Power supply"
- note added: "replace to ACS711 for 3.3v use."
- note added: "replace to AT25F512B for 5v use."
- note added: "to use 3.3v on all devices"
- moved on the sheet: C1, C10, C2, C3, C4, C5, D1, IC1, IC3, IC5, IC7, L1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
